Commit message: Finish wrist markers and pin material-preserving platform asset
Signed-off-by: Mohammed Magdy <mohamed@botshare.ai>

File: ros2/src/openamrobot_upperbody_description/urdf/upper_sensors.xacro (robot description, xacro)
@@ -27,4 +27,6 @@
     <link name="${name}_link">
       <visual>
+        <!-- Existing dark equipment finish; this remains a provisional frame marker. -->
+        <material name="equipment_black"><color rgba="0.035 0.045 0.055 1"/></material>
         <geometry><box size="${openamr_sensor_marker_edge} ${openamr_sensor_marker_edge} ${openamr_sensor_marker_edge}"/></geometry>
       </visual>
