Commit message: Support the head camera visually and close simulation lifecycle races
Signed-off-by: Mohammed Magdy <mohamed@botshare.ai>

File: ros2/src/openamrobot_upperbody_description/urdf/openamrobot_upperbody.xacro (robot description, xacro)
@@ -70,19 +70,16 @@
     <xacro:property name="lens" value="${geo['head_camera_lens']}" lazy_eval="false"/>
     <xacro:property name="profile" value="${geo['arm_profile']}" lazy_eval="false"/>
-    <!-- Presentation only, not a datum: one colour for every placeholder box. -->
-    <xacro:property name="placeholder_rgba" value="0.78 0.64 0.45 1.0" lazy_eval="false"/>
-    <material name="placeholder_geometry">
-      <color rgba="${placeholder_rgba}"/>
-    </material>
-    <xacro:macro name="openamrobot_placeholder_gazebo_material" params="link">
-      <gazebo reference="${link}">
-        <visual>
-          <material>
-            <ambient>${placeholder_rgba}</ambient>
-            <diffuse>${placeholder_rgba}</diffuse>
-            <specular>0.1 0.1 0.1 1.0</specular>
-          </material>
-        </visual>
-      </gazebo>
+    <!-- Presentation only: neutral reference finishes do not assert released hardware geometry.
+         Material names are shared by the URDF and Gazebo extensions. -->
+    <xacro:property name="openamr_finishes" value="${dict(structural_aluminum='0.63 0.67 0.71 1', adapter_gray='0.25 0.28 0.31 1', equipment_black='0.035 0.045 0.055 1', equipment_metal='0.45 0.48 0.52 1', sensor_dark='0.09 0.10 0.11 1', estop_red='0.80 0.025 0.025 1', flag_steel='0.20 0.22 0.25 1')}"/>
+    <xacro:macro name="openamr_finish" params="material">
+      <material name="${material}"><color rgba="${openamr_finishes[material]}"/></material>
+    </xacro:macro>
+    <xacro:macro name="openamr_gazebo_finish" params="link material">
+      <gazebo reference="${link}"><visual><material>
+        <ambient>${openamr_finishes[material]}</ambient>
+        <diffuse>${openamr_finishes[material]}</diffuse>
+        <specular>0.15 0.15 0.15 1</specular>
+      </material></visual></gazebo>
     </xacro:macro>
     <!-- Column axis on the base-plate top face (height reference, 304 mm). -->
@@ -99,5 +96,5 @@
           <origin xyz="0 0 ${col['retracted_length'] / 2}" rpy="0 0 0"/>
           <geometry><box size="${column_geometry['section_x']} ${column_geometry['section_y']} ${col['retracted_length']}"/></geometry>
-          <material name="placeholder_geometry"/>
+          <xacro:openamr_finish material="structural_aluminum"/>
         </visual>
         <collision name="placeholder_lift_column_fixed_stage">
@@ -108,5 +105,5 @@
     </link>
     <xacro:unless value="${column_geometry == ''}">
-      <xacro:openamrobot_placeholder_gazebo_material link="lift_column_base_link"/>
+      <xacro:openamr_gazebo_finish material="structural_aluminum" link="lift_column_base_link"/>
     </xacro:unless>
     <joint name="lift_column_base_joint" type="fixed">
@@ -126,5 +123,5 @@
           <origin xyz="0 0 ${-col['stroke'] / 2}" rpy="0 0 0"/>
           <geometry><box size="${column_geometry['inner_x']} ${column_geometry['inner_y']} ${col['stroke']}"/></geometry>
-          <material name="placeholder_geometry"/>
+          <xacro:openamr_finish material="structural_aluminum"/>
         </visual>
         <collision name="placeholder_lift_column_moving_stage">
@@ -133,5 +130,5 @@
         </collision>
       </link>
-      <xacro:openamrobot_placeholder_gazebo_material link="lift_carriage_link"/>
+      <xacro:openamr_gazebo_finish material="structural_aluminum" link="lift_carriage_link"/>
     </xacro:unless>
     <joint name="lift_joint" type="prismatic">
@@ -149,5 +146,5 @@
         <visual>
           <geometry><box size="${adapter_plate['size_x']} ${adapter_plate['size_y']} ${geo['adapter_plate_thickness']}"/></geometry>
-          <material name="placeholder_geometry"/>
+          <xacro:openamr_finish material="adapter_gray"/>
         </visual>
         <collision name="adapter_plate">
@@ -155,5 +152,5 @@
         </collision>
       </link>
-      <xacro:openamrobot_placeholder_gazebo_material link="adapter_plate_link"/>
+      <xacro:openamr_gazebo_finish material="adapter_gray" link="adapter_plate_link"/>
       <joint name="adapter_plate_joint" type="fixed">
         <parent link="lift_carriage_link"/>
@@ -166,5 +163,5 @@
       <visual>
         <geometry><box size="${profile['size_x']} ${profile['size_y']} ${profile['length']}"/></geometry>
-        <material name="placeholder_geometry"/>
+        <xacro:openamr_finish material="structural_aluminum"/>
       </visual>
       <collision>
@@ -172,5 +169,5 @@
       </collision>
     </link>
-    <xacro:openamrobot_placeholder_gazebo_material link="arm_profile_link"/>
+    <xacro:openamr_gazebo_finish material="structural_aluminum" link="arm_profile_link"/>
     <!-- With the adapter plate modelled the profile hangs off the plate it stands on (P28): the two faces touch by design (the profile's bottom
          face is the plate's top face), and two siblings that touch would be a permanent collision of the model, where a parent and its child are
@@ -205,5 +202,31 @@
     <!-- Head camera (ZED Mini). head_camera_mount_link is the pitch pivot on the
          lens line; head_camera_link is pitched down by head_pitch about y. -->
-    <link name="head_camera_mount_link"/>
+    <!-- Provisional VISUAL-ONLY camera support, from the assembled roadmap's
+         head_camera_bracket (model.js cd780d6368625f4c653dfa287efc0688c37be82a).
+         Released bracket CAD is pending (upperbody-hw upper_body_option_B.md).
+         It adds no link/joint, mass, inertia or collision; its fixed camera-mount
+         frame is already carried by the lift. The camera pivot/optical pose is unchanged. -->
+    <!-- Visualization constant: roadmap support footprint/width, not a released bracket dimension. -->
+    <xacro:property name="openamr_head_support_width" value="0.030"/>
+    <!-- Visualization constant: roadmap foot thickness, visual only. -->
+    <xacro:property name="openamr_head_support_foot" value="0.006"/>
+    <!-- Visualization constant: roadmap stem depth, visual only. -->
+    <xacro:property name="openamr_head_support_depth" value="0.012"/>
+    <!-- Visualization constant: roadmap setback behind the lens line, visual only. -->
+    <xacro:property name="openamr_head_support_setback" value="0.030"/>
+    <xacro:property name="head_support_rise" value="${mount['z_above_column_top'] + lens['z_above_arm_mount'] - geo['adapter_plate_thickness'] - profile['length']}"/>
+    <link name="head_camera_mount_link">
+      <visual>
+        <origin xyz="${-openamr_head_support_setback} 0 ${-head_support_rise + openamr_head_support_foot/2}"/>
+        <geometry><box size="${openamr_head_support_width} ${openamr_head_support_width} ${openamr_head_support_foot}"/></geometry>
+        <xacro:openamr_finish material="structural_aluminum"/>
+      </visual>
+      <visual>
+        <origin xyz="${-openamr_head_support_setback} 0 ${-head_support_rise/2}"/>
+        <geometry><box size="${openamr_head_support_depth} ${openamr_head_support_width} ${head_support_rise}"/></geometry>
+        <xacro:openamr_finish material="structural_aluminum"/>
+      </visual>
+    </link>
+    <xacro:openamr_gazebo_finish link="head_camera_mount_link" material="structural_aluminum"/>
     <joint name="head_camera_mount_joint" type="fixed">
       <parent link="lift_carriage_link"/>

File: ros2/src/openamrobot_upperbody_description/urdf/upper_body_equipment.xacro (robot description, xacro)
@@ -6,5 +6,5 @@
   CHEST-JSON and LIFT-JSON, chestItems() and liftSensors()), with selected supplier envelope corrections recorded in datums.yaml.
   Placeholders until work package M-09.
-  Geometry only: fixed joints, boxes and cylinders, the column's placeholder material. No logic, no ros2_control, no topics,
+  Geometry only: fixed joints, boxes and cylinders, neutral visual materials. No logic, no ros2_control, no topics,
   no command authority. The second E-stop and the lift-stop sensors are drawn here as volumes; nothing here reads, wires or
   acts on them.
@@ -33,11 +33,10 @@
     </inertial>
   </xacro:macro>
-  <!-- A box as visual and collision, at xyz in the link. Only the collision is named: sdformat applies the link's <gazebo> material block
-       only to unnamed visuals (test_p25_placeholder_material). -->
-  <xacro:macro name="openamrobot_equipment_box" params="name size xyz">
-    <visual>
+  <!-- Existing box geometry/pose/collision is unchanged. Named visuals retain their individual URDF finish through SDFormat conversion; no link-wide override recolours the red actuator or dark sensor bodies. -->
+  <xacro:macro name="openamrobot_equipment_box" params="name size xyz material:=structural_aluminum">
+    <visual name="${name}">
       <origin xyz="${xyz[0]} ${xyz[1]} ${xyz[2]}" rpy="0 0 0"/>
       <geometry><box size="${size[0]} ${size[1]} ${size[2]}"/></geometry>
-      <material name="placeholder_geometry"/>
+      <xacro:openamr_finish material="${material}"/>
     </visual>
     <collision name="${name}">
@@ -62,7 +61,6 @@
     <link name="getac_tablet_link">
       <xacro:openamrobot_equipment_box_inertial mass="${eq['getac_tablet_mass']['value']}" size="${tablet}"/>
-      <xacro:openamrobot_equipment_box name="placeholder_getac_tablet" size="${tablet}" xyz="${[0, 0, 0]}"/>
+      <xacro:openamrobot_equipment_box name="placeholder_getac_tablet" material="equipment_black" size="${tablet}" xyz="${[0, 0, 0]}"/>
     </link>
-    <xacro:openamrobot_placeholder_gazebo_material link="getac_tablet_link"/>
     <joint name="getac_tablet_joint" type="fixed">
       <parent link="arm_profile_link"/>
@@ -72,7 +70,6 @@
     <link name="head_light_link">
       <xacro:openamrobot_equipment_box_inertial mass="${eq['head_light_mass']['value']}" size="${light}"/>
-      <xacro:openamrobot_equipment_box name="placeholder_head_light" size="${light}" xyz="${[0, 0, 0]}"/>
+      <xacro:openamrobot_equipment_box name="placeholder_head_light" material="equipment_metal" size="${light}" xyz="${[0, 0, 0]}"/>
     </link>
-    <xacro:openamrobot_placeholder_gazebo_material link="head_light_link"/>
     <joint name="head_light_joint" type="fixed">
       <parent link="arm_profile_link"/>
@@ -86,12 +83,11 @@
     <xacro:property name="es_head" lazy_eval="false" value="${eq['second_estop_head_size']['value']}"/>
     <link name="second_estop_link">
-      <xacro:openamrobot_equipment_box name="placeholder_second_estop_contact_block" size="${es_block}"
+      <xacro:openamrobot_equipment_box name="placeholder_second_estop_contact_block" material="equipment_black" size="${es_block}"
                                        xyz="${[-panel_behind + es_block[0] / 2, 0, 0]}"/>
-      <xacro:openamrobot_equipment_box name="placeholder_second_estop_collar" size="${es_collar}"
+      <xacro:openamrobot_equipment_box name="placeholder_second_estop_collar" material="equipment_metal" size="${es_collar}"
                                        xyz="${[-panel_behind + es_block[0] + es_collar[0] / 2, 0, 0]}"/>
-      <xacro:openamrobot_equipment_box name="placeholder_second_estop_head" size="${es_head}"
+      <xacro:openamrobot_equipment_box name="placeholder_second_estop_head" material="estop_red" size="${es_head}"
                                        xyz="${[-panel_behind + es_block[0] + es_collar[0] + es_head[0] / 2, 0, 0]}"/>
     </link>
-    <xacro:openamrobot_placeholder_gazebo_material link="second_estop_link"/>
     <joint name="second_estop_joint" type="fixed">
       <parent link="lift_column_base_link"/>
@@ -110,8 +106,8 @@
     <xacro:macro name="openamrobot_lift_stop_sensor" params="stop z">
       <link name="lift_stop_sensor_${stop}_link">
-        <visual>
+        <visual name="lift_stop_sensor_body">
           <origin xyz="${s_len / 2} 0 0" rpy="0 ${pi / 2} 0"/>
           <geometry><cylinder radius="${eq['lift_stop_sensor_diameter']['value'] / 2}" length="${s_len}"/></geometry>
-          <material name="placeholder_geometry"/>
+          <xacro:openamr_finish material="sensor_dark"/>
         </visual>
         <collision name="placeholder_lift_stop_sensor">
@@ -138,5 +134,4 @@
             size="${[b_t,span/2-hy-bore/2,bore]}" xyz="${[b_x-b_t/2,cy+(span/2+hy+bore/2)/2,0]}"/>
       </link>
-      <xacro:openamrobot_placeholder_gazebo_material link="lift_stop_sensor_${stop}_link"/>
       <joint name="lift_stop_sensor_${stop}_joint" type="fixed">
         <parent link="lift_column_base_link"/>
@@ -166,5 +161,4 @@
           size="${[rod_w,rod_w,ct]}" xyz="${[0,-rod_w,-ct/2]}"/>
     </link>
-    <xacro:openamrobot_placeholder_gazebo_material link="lift_flag_rod_link"/>
     <joint name="lift_flag_rod_joint" type="fixed">
       <parent link="adapter_plate_link"/>
@@ -174,7 +168,6 @@
     </joint>
     <link name="lift_flag_link">
-      <xacro:openamrobot_equipment_box name="placeholder_lift_flag" size="${flag}" xyz="${[0, 0, 0]}"/>
+      <xacro:openamrobot_equipment_box name="placeholder_lift_flag" material="flag_steel" size="${flag}" xyz="${[0, 0, 0]}"/>
     </link>
-    <xacro:openamrobot_placeholder_gazebo_material link="lift_flag_link"/>
     <joint name="lift_flag_joint" type="fixed">
       <parent link="lift_flag_rod_link"/>

Commit message: description: ZED Mini body on head_camera_link and the OpenArm mount placeholder
The head camera had frames and no body. head_camera_link (option B's frame on
the lens line, pitched by head_pitch) now carries a ZED Mini box, visual and
collision, and its mass, when the combined robot passes the datums; the
standalone model keeps a bare frame. head_camera_bracket_link (child of the
geometry-free lens pivot head_camera_mount_link) is a placeholder for the
OpenArm-supplied mount: a foot plate on the arm-profile top and a post up to the
lens line, as the docs model draws it.

Datums (revision 2026-11-01.b): head_camera_size [0.0265, 0.1245, 0.0305] and
head_camera_mass 0.0629 (supplier, provisional: Stereolabs datasheet 124.5 x
30.5 x 26.5 mm, 62.9 g; URLs in ref; NOT read first-hand, the Stereolabs hosts
are blocked by this session's network policy, values from a search summary);
head_camera_body_x_from_lens_line -0.013 and head_camera_bracket_* (placeholder,
"not stated": the mount has no published dimensions; values as model.js draws
them). Recorded discrepancy: Stereolabs zed_description gives the ZED Mini
height as 0.0265 (its mesh 29.5 x 125.2 x 26.6 mm), the docs model draws 30.5
tall and 26.5 deep; the docs assignment is kept so the two models agree.

Tests: the body sits at the HEAD-CAMERA-IDENTITY pose (lens 0.042 ahead of and
0.223 above the arm mount, centred, hp30) and pitches with hp15/hp35; the mount
runs from the profile top to the lens line; T12 asserts the three new lists;
export_docs_model_values.py gains a HEAD-CAMERA block read from the URDF, and
docs_head_camera() reads the same values from model.js source (fixture: the
verbatim lines of docs cd780d6, hash-checked); live comparison: equal.
Reverts fail: body removed 8 failed; body collision renamed 8 failed; lens
0.042 -> 0.022 6 failed; body x -0.013 -> -0.015 fails the docs comparison.

Consequences, updated with a reason in each test: E01's top is now the body's
rear top edge, 1.5993 m (was the lens frame, 1.573; limit 1.700 unchanged);
P25 lists the two new placeholder-material users; the collision matrix is
re-derived: 179 -> 198 pairs (20 + 29 Adjacent + 149 ConstantTransform; 19
added, none removed or relabelled, no constant pair colliding), tallies updated
with a history line. The arm collision report covers the two new links.

Signed-off-by: Alex Reznichenko <info@botshare.ai>
Assisted-by: Claude Code

File: ros2/src/openamrobot_upperbody_description/urdf/openamrobot_upperbody.xacro (robot description, xacro)
@@ -211,5 +211,14 @@
       <origin xyz="${mount['x_from_column_axis'] + lens['x_ahead_of_arm_mount']} ${lens['y']} ${mount['z_above_column_top'] + lens['z_above_arm_mount']}" rpy="0 0 0"/>
     </joint>
-    <link name="head_camera_link"/>
+    <!-- With the datums (combined robot): the ZED Mini body (upper_body_equipment.xacro); without: a frame, as before. -->
+    <xacro:if value="${datums == ''}">
+      <link name="head_camera_link"/>
+    </xacro:if>
+    <xacro:unless value="${datums == ''}">
+      <link name="head_camera_link">
+        <xacro:openamrobot_head_camera_body datums="${datums}"/>
+      </link>
+      <xacro:openamrobot_placeholder_gazebo_material link="head_camera_link"/>
+    </xacro:unless>
     <joint name="head_camera_pitch_joint" type="fixed">
       <parent link="head_camera_mount_link"/>

File: ros2/src/openamrobot_upperbody_description/urdf/upper_body_equipment.xacro (robot description, xacro)
@@ -14,4 +14,6 @@
       arm_profile_link  -> getac_tablet_link       Getac ZX80, landscape, screen forward, rear face on the profile front face
                         -> head_light_link         Falcon FLDL-i150x15-W, top edge head_light_gap_below_tablet below the tablet
+      head_camera_link (option B's frame)          Stereolabs ZED Mini body box, pitched with the frame
+      head_camera_mount_link -> head_camera_bracket_link   placeholder for the OpenArm-supplied mount, profile top to lens line
       adapter_plate_link -> lift_flag_rod_link     MISUMI 20 x 20 rod hanging from the plate underside (frame at its top end)
                             -> lift_flag_link      SS400 flag, lift_flag_gap from the sensor faces
@@ -45,4 +47,20 @@
       <geometry><box size="${size[0]} ${size[1]} ${size[2]}"/></geometry>
     </collision>
+  </xacro:macro>
+  <!-- Stereolabs ZED Mini body on head_camera_link (option B's frame on the lens line, pitched by head_pitch), so the box pitches with it:
+       datums head_camera_size (x along the optical axis, y across, z up in head_camera_link), head_camera_body_x_from_lens_line, head_camera_mass.
+       Called by openamrobot_upperbody.xacro inside its head_camera_link when the combined robot passes the datums. -->
+  <xacro:macro name="openamrobot_head_camera_body" params="datums">
+    <xacro:property name="cam" lazy_eval="false" value="${datums['datums']['head_camera_size']['value']}"/>
+    <xacro:property name="cam_x" lazy_eval="false" value="${datums['datums']['head_camera_body_x_from_lens_line']['value']}"/>
+    <xacro:property name="cam_m" lazy_eval="false" value="${datums['datums']['head_camera_mass']['value']}"/>
+    <inertial>
+      <origin xyz="${cam_x} 0 0" rpy="0 0 0"/>
+      <mass value="${cam_m}"/>
+      <inertia ixx="${cam_m * (cam[1] * cam[1] + cam[2] * cam[2]) / 12}" ixy="0" ixz="0"
+               iyy="${cam_m * (cam[0] * cam[0] + cam[2] * cam[2]) / 12}" iyz="0"
+               izz="${cam_m * (cam[0] * cam[0] + cam[1] * cam[1]) / 12}"/>
+    </inertial>
+    <xacro:openamrobot_equipment_box name="placeholder_head_camera_body" size="${cam}" xyz="${[cam_x, 0, 0]}"/>
   </xacro:macro>
   <xacro:macro name="openamrobot_upper_body_equipment" params="datums col geo">
@@ -135,4 +153,24 @@
     <xacro:openamrobot_lift_stop_sensor stop="l1175" z="${eq['lift_stop_sensor_z_l1175']['value']}"/>
     <xacro:openamrobot_lift_stop_sensor stop="l1350" z="${eq['lift_stop_sensor_z_l1350']['value']}"/>
+    <!-- ===== Head camera mount (moving): placeholder for the OpenArm-supplied mount between the camera and the arm-profile top. Its
+         dimensions are not stated by any supplier; the values are the docs model's drawing (datums head_camera_bracket_*, placeholder). A foot
+         plate on the profile top and a post up to the lens line. It hangs from head_camera_mount_link (the pivot on the lens line, no geometry),
+         so it is the camera body's structural neighbour: the drawn post reaches into the pitched body. Frame: foot plate underside centre. ===== -->
+    <xacro:property name="arm_mount" lazy_eval="false" value="${geo['arm_mount']}"/>
+    <xacro:property name="lens_z" lazy_eval="false" value="${arm_mount['z_above_column_top'] + geo['head_camera_lens']['z_above_arm_mount']}"/>
+    <xacro:property name="profile_top" lazy_eval="false" value="${plate_t + profile['length']}"/>
+    <xacro:property name="foot" lazy_eval="false" value="${eq['head_camera_bracket_foot_size']['value']}"/>
+    <xacro:property name="post" lazy_eval="false" value="${eq['head_camera_bracket_post_section']['value']}"/>
+    <link name="head_camera_bracket_link">
+      <xacro:openamrobot_equipment_box name="placeholder_head_camera_bracket_foot" size="${foot}" xyz="${[0, 0, foot[2] / 2]}"/>
+      <xacro:openamrobot_equipment_box name="placeholder_head_camera_bracket_post" size="${[post[0], post[1], lens_z - profile_top]}"
+                                       xyz="${[0, 0, (lens_z - profile_top) / 2]}"/>
+    </link>
+    <xacro:openamrobot_placeholder_gazebo_material link="head_camera_bracket_link"/>
+    <joint name="head_camera_bracket_joint" type="fixed">
+      <parent link="head_camera_mount_link"/>
+      <child link="head_camera_bracket_link"/>
+      <origin xyz="${-eq['head_camera_bracket_x_behind_lens']['value']} 0 ${profile_top - lens_z}" rpy="0 0 0"/>
+    </joint>
     <!-- ===== Flag rod and flag (moving), hanging from the adapter plate underside ===== -->
     <xacro:property name="flag" lazy_eval="false" value="${eq['lift_flag_size']['value']}"/>
