Commit message: description: item 24 upper-body equipment, same as the docs model (#26)
* feat(description): canonical combined description, mast macro and expansion tests

Add the openamrobot_upperbody_description package content for A6 (part of #7):

- urdf/combined_robot.xacro: base (platform-sw, included unchanged) + mast +
  two upstream openarm_v20_robot calls (ADR-008, no OpenArm body). Args
  mast_id, arm_package, hardware_profile, enable_planar_base, datums_file;
  an unknown value fails expansion via xacro.fatal with the accepted list.
- urdf/mast.xacro: openamr_mast macro; mast_offset per corrected ADR-006
  (shoulder_height - base_link_height_above_floor - mast_base_pose.z -
  left_arm_mount_pose.z); no upstream body reference point is read.
- config: datums.yaml (schema v1, revision 2026-10-08.a), mast_ids.yaml (four
  IDs, default mast_1350), frame_contract.yaml, and left/right OpenArm presets
  derived from openarm_description @ 14ff67b (Apache-2.0, two lines changed).
- launch/view.launch.py with RViz config.
- test: T01 (mast_id x arm_package expansion), T03 (one root, no duplicates),
  T06 (arg validation).

ros2_control, sensors and the planar joint are not emitted yet;
hardware_profile and enable_planar_base are validated only.

Assisted-by: Claude Code
Signed-off-by: Tushar Goel <Slash8860300674@gmail.com>

* feat(description): datum schema, reference checks and mast-height tests

Add the S3 checks for openamrobot_upperbody_description (part of #7):

- config/datums.schema.json (JSON Schema 2020-12): required provenance
  fields, source/status enums, verified => evidenced source + non-empty ref,
  source placeholder => status placeholder, top-level report_only and
  pending_reference.
- datums.yaml: new pending_reference map (head and wrist camera poses ->
  S4); revision 2026-10-08.b because the file content changed.
- T12: datums.yaml validates; test/fixtures/datums_broken.yaml is rejected
  and every rule is shown to bite on its own.
- T13: every datums[...] key in urdf/*.xacro exists, parsed from the xacro
  text; every datum is in exactly one of referenced / report_only /
  pending_reference; a pending entry whose consumer exists fails.
- T05: floor-relative height of openarm_{left,right}_base_link equals
  shoulder_height for all four mast IDs (+-1 mm), also with the placeholders
  moved. Left and right plate z must be equal. The xacro must not read
  body/struct/reference_points or 0.698.
- test/urdf_utils.py: fixed-joint FK helper (numpy) with its own tests.
- scripts/datums_report.py: datums by status and source, placeholder list.
- Revision guard: datums.yaml content must not change vs HEAD~ without a
  revision change (skips outside a git checkout).
- W01 (WARN): base_link inertia is not seen by KDL consumers. Recorded, not
  fixed (ADR-005).

Assisted-by: Claude Code
Signed-off-by: Tushar Goel <Slash8860300674@gmail.com>

* feat(description): upper-body sensor frames, planar base joint and enforced frame contract

Add the S4 content of openamrobot_upperbody_description (part of #7):

- urdf/upper_sensors.xacro, emitted for arm_package == openarm: head camera
  on mast_mount_link and a wrist camera on each openarm_*_ee_base_link, each
  with a REP-103 optical frame, poses from the head/wrist camera datums.
  Marker-box visual only: no collision, no inertial (collision_free: true in
  the frame contract, with the reason). Plain frames; the ZED wrapper stays
  deferred.
- SO-101 stub: so101_mount_joint/link at identity on mast_mount_link; A9 owns
  everything below it.
- Planar base joint, emitted only with enable_planar_base:=true, under the
  A6 comment (disabled by default, AD-30): world link + base_planar_joint
  (planar, world -> base_link, axis z). The arg quoting in
  combined_robot.xacro is unchanged and now guarded by a test.
- frame_contract.yaml: base_link gets `variants` (root by default, planar
  child of world with enable_planar_base == true) so the contract is right
  in every expansion; collision_free fields on the three camera links.
- datums.yaml: the three pending_reference entries are deleted in this
  commit, which references those datums; revision 2026-10-08.c.
- T04: every expansion of the T01 matrix plus the planar flag honours the
  contract (R/C/W, parent and type, unlisted frames in our namespaces fail),
  missing W frames go to a JSON sidecar as a WARN. The checker is tested on
  synthetic URDFs.
- T11: no world/planar joint by default; correct when enabled; comment block
  present in the source. Sensor and so101 stub tests.
- view.launch.py gains enable_planar_base.

ros2_control is not emitted yet.

Assisted-by: Claude Code
Signed-off-by: Tushar Goel <Slash8860300674@gmail.com>

* feat(description): A6 evidence checks, config id and verify_a6.sh

Add the S5 verification for openamrobot_upperbody_description (part of #7):

- T02: check_urdf on the 12 T01 expansions plus openarm on gazebo and real
  at mast_1350, and the planar-flag expansions (extra, labelled). A missing
  check_urdf is a FAIL, not a skip.
- T07/T08: every link with an inertial or visual has a collision or is
  collision_free with a reason (FAIL); collision mesh == visual mesh is
  listed (WARN only).
- T09: mass > 0, Ixx/Iyy/Izz > 0, principal moments > 0, triangle
  inequality, tensor positive-definite (numpy eigenvalues).
- T10: modelled mass by owner (base, mast, openarm_*, sensors), the not
  modelled list in words, the W01 line; FAIL only above gross_mass_limit.
- E01: approximate assembled height (zero pose, frame origins and
  box/cylinder/sphere extents, no mesh extents) against max_assembled_height;
  WARN for analysis mast IDs, FAIL for the release one.
- W02 (WARN): KDL converts base_planar_joint to a fixed joint. Observed from
  a real robot_state_publisher; recorded as a consumer limitation that does
  not affect A6 acceptance. Planar base motion for A7 comes from Gazebo's
  odom -> base_link, never from robot_state_publisher.
- scripts/print_config_id.py: full sha256:<64 hex> over the canonical
  expanded URDF, mast_id, arm_package, hardware_profile, datums.revision and
  the pinned openarm_description commit. C01 asserts the format and
  validates it against the pattern in the installed C9 schema (SKIP with the
  reason if openamrobot-interfaces is not in the workspace).
- Evidence directory: default is now <workspace>/evidence, found from the
  package share path; OPENAMR_EVIDENCE_DIR overrides; never a temp dir (T04's
  sidecar moves with it).
- T13: visualization constants (DATUMS.md) must be visual-only, a named
  property with a comment saying so, and are listed in the evidence. The
  comment on openamr_sensor_marker_edge now says it; the expansion is
  unchanged.
- scripts/verify_a6.sh runs colcon test, the T02 matrix, datums_report.py
  and the config ids, and writes evidence/<UTC ts>_dev.json
  (evidence_class static+mock). Exit status is non-zero iff any check is FAIL.
  T14-T16 and L01 are SKIP (S7), not passed.

Assisted-by: Claude Code
Signed-off-by: Tushar Goel <Slash8860300674@gmail.com>

* docs(description): Layer-1 README for the canonical description package

Args, how to build, view and verify, adding a mast ID or arm package, the datum rules and the known limitations.

Assisted-by: Claude Code
Signed-off-by: Tushar Goel <Slash8860300674@gmail.com>

* docs: state the scaffold status of the control, bringup, gazebo and moveit packages

Each README says what is not implemented, what is intended, and where the model can be viewed today.

Assisted-by: Claude Code
Signed-off-by: Tushar Goel <Slash8860300674@gmail.com>

* docs: point the README at the description package, add CHANGELOG, remove config/lift

config/lift/ was an empty scaffold directory; an actuated lift is OpenAMRobot 3.0 scope. The mast configuration text is unchanged.

Assisted-by: Claude Code
Signed-off-by: Tushar Goel <Slash8860300674@gmail.com>

* fix(description): mast_section is the MISUMI HFS6-60120 profile, 60 x 120 mm

The datum held an invented 80 mm square marked placeholder. The profile is
named in this repo's README and in P-03 rev 18.2, and in MISUMI's HFS
nomenclature the suffix is the cross-section in mm. Set [0.060, 0.120],
source plan, status provisional: the part number gives the section but not
which axis carries the 120 mm (x fore-aft / y lateral is assumed, because it
puts the side faces at y = +/-0.060 where the J1_A plates already sit).

Revision 2026-10-08.c -> .d; every config_id changes, legitimately, because
the revision is an input. README datum counts updated (8 placeholder,
5 provisional, 1 verified).

Assisted-by: Claude Code
Signed-off-by: Tushar Goel <Slash8860300674@gmail.com>

* feat(description): arm ros2_control profiles for mock, gazebo and real

urdf/ros2_control.xacro defines openamr_arm_ros2_control(hardware_profile),
called from combined_robot.xacro for arm_package:=openarm only. The base never
gets a <ros2_control> block (ADR-003).

- mock and real call upstream openarm_bimanual_ros2_control as upstream's own
  top-level v2.0 file does (same gains file, same finger-mimic file, same
  prefixes); use_fake_hardware follows the profile. The two blocks are equal,
  whitespace aside, to that file's expansion, and T14 and T16 assert it.
- gazebo emits our own system block, gz_ros2_control/GazeboSimSystem, for the
  same joints and the same command and state interfaces the upstream macro
  declares. finger_joint2 is left out as upstream leaves it out; whether
  gz_ros2_control needs a mimic parameter there is a TODO.

hardware_profile no longer prints "no effect yet" for a non-mock value.

T14 (mock: GenericSystem, no OpenArmHW, no base ros2_control, JTC interfaces
exported), T15 (gazebo) and T16 (real: OpenArmHW and CAN parameters, gains from
the upstream file) are expansion checks.

Assisted-by: Claude Code
Signed-off-by: Tushar Goel <Slash8860300674@gmail.com>

* feat(control): arm_controllers.yaml for both arms, one file for every profile

controller_manager at 100 Hz; joint_state_broadcaster; left and right arm
controllers (JointTrajectoryController, joints 1-7, position command,
position and velocity state); left and right gripper controllers
(position_controllers/GripperActionController on finger_joint1).

Derived from enactic/openarm_ros2 ros2_controllers.yaml @ 4e837e1 with an
attribution header. Changes from upstream: arm state interfaces drop effort;
the gripper controllers name their joint with `joint:` because the Jazzy
GripperActionController reads that and fails to configure ("Joint name cannot
be empty") on upstream's `joints:` list.

test_arm_controllers_yaml.py checks every joint the YAML names against the
<ros2_control> blocks of the mock, gazebo and real expansions, that every
declared joint has exactly one controller, and that the finger_joint2 mimic has
none.

Assisted-by: Claude Code
Signed-off-by: Tushar Goel <Slash8860300674@gmail.com>

* feat(bringup): mock bringup with all five controllers; view.launch.py moves here

mock.launch.py starts robot_state_publisher on the combined description with
hardware_profile:=mock, ros2_control_node with
openamrobot_upperbody_control/config/arm_controllers.yaml, and spawners for
joint_state_broadcaster, left_arm_controller, right_arm_controller,
left_gripper_controller and right_gripper_controller. Args: mast_id, rviz
(default false). The base is not started.

L01 (launch_testing, own random ROS_DOMAIN_ID, localhost only) starts it
headless, waits up to 30 s for all five controllers to be active through
/controller_manager/list_controllers, sends one FollowJointTrajectory goal to
left_arm_controller and asserts /joint_states reaches the target within 0.02 rad
with the right arm unmoved, then that every process exits cleanly.

view.launch.py moves from the description package to bringup (no forwarder: it
would make description depend on bringup). The description package drops its
launch/ install directory and the launch, launch_ros, rviz2 and
joint_state_publisher_gui depends, which went with the file.

Assisted-by: Claude Code
Signed-off-by: Tushar Goel <Slash8860300674@gmail.com>

* feat(description): report T14-T16 and L01 as results, not SKIPs

build_evidence.py no longer lists T14, T15, T16 and L01 as not implemented: a
check with no result is a FAIL again. L01 is a launch test in
openamrobot_upperbody_bringup, so the report now reads that package's xunit
directory too (read_xunit_dirs, counts for one ID add up, stale-file handling is
unchanged) and verify_a6.sh runs the tests of the control and bringup packages
next to its own. The limitations list says what the new checks do not cover: no
Gazebo or real plugin is loaded, the finger_joint2 mimic under gz_ros2_control is
a TODO, and mock hardware reflects commands as state.

NOT_IMPLEMENTED stays as an empty mechanism, tested with a monkeypatched entry.

Assisted-by: Claude Code
Signed-off-by: Tushar Goel <Slash8860300674@gmail.com>

* docs: describe the arm ros2_control profiles, the controllers and the mock bringup

Description README: hardware_profile now selects the arm plugin, a ros2_control
section, T14-T16 and L01 in the check table instead of SKIP, the new known
limitation (verified on mock only), and view.launch.py's new home. Control and
bringup READMEs replace the scaffold text; the bringup README documents the mock
launch and a trajectory command that was run against it.

Assisted-by: Claude Code
Signed-off-by: Tushar Goel <Slash8860300674@gmail.com>

* fix: package.xml descriptions of bringup, control and moveit state the 2.0 fixed-mast scope

The three descriptions still said "lift" (issue #7). They now say what the
packages are for OpenAMRobot 2.0: a fixed mast and two OpenArm v2.0 arms, in the
description package's wording. The README sentences that excused the stale
strings are removed. The moveit description says it is a scaffold, which it is.

Refs #7.

Assisted-by: Claude Code
Signed-off-by: Tushar Goel <Slash8860300674@gmail.com>

* docs: bring CHANGELOG current with the ros2_control profiles and the mast_section fix

It still said T14-T16 and L01 were SKIP, hardware_profile had no effect, and
view.launch.py lived in the description package. Adds the P06 entries (profiles,
controllers, mock bringup, L01), the mast_section datum change and the datum
counts, and the corrected package descriptions. The known-limitations list now
says ros2_control is runtime-verified on mock only.

Assisted-by: Claude Code
Signed-off-by: Tushar Goel <Slash8860300674@gmail.com>

* chore: keep shell scripts on LF line endings (.gitattributes)

This checkout is edited through /mnt/c; a shell script that picks up CRLF fails
with "\r: command not found", and verify_a6.sh is shipped and run through
`ros2 run`. Line endings are a repository-wide property, so the rule is at the
root. Renormalising changes nothing: verify_a6.sh is already LF in the index and
the working tree.

Assisted-by: Claude Code
Signed-off-by: Tushar Goel <Slash8860300674@gmail.com>

* docs(control): the gripper controller's replacement changes the action interface

position_controllers/GripperActionController is deprecated in Jazzy, but its
replacement, parallel_gripper_action_controller/GripperActionController, is not
the same controller under a new name: it serves
control_msgs/action/ParallelGripperCommand, the deprecated one serves
control_msgs/action/GripperCommand (what upstream's MoveIt configuration
expects). Read from the Jazzy 4.42 libraries and observed live.

The type therefore stays as it is, and the README says why: switching would
decide manipulation#11 / ADR-009 point 4, which is open with Om and Adnan.

Assisted-by: Claude Code
Signed-off-by: Tushar Goel <Slash8860300674@gmail.com>

* feat(description): config id falls back to a pinned upstream commit when there is no checkout

print_config_id.py read the openarm_description commit from the git checkout only
and failed without one, so a CI machine or an installed package without sources
could not produce an id. config/upstream_pins.yaml now carries the pin; the git
checkout still wins, a checkout with local changes is still an error (never
replaced by the pin, which would hide the change), and the report's limitations
say when the commit came from the metadata. --explain names the source.

The constant cannot rot unnoticed: test_c01 fails if it disagrees with the
checkout or with the openamrobot-manipulation baseline pin, and checks that the
fallback gives the same id as the checkout.

Assisted-by: Claude Code
Signed-off-by: Tushar Goel <Slash8860300674@gmail.com>

* feat(description): T02 also runs check_urdf on gazebo and real at mast_1300

The T01 matrix has the other profiles at the release mast_id only, which is what
VERIFICATION.md specifies and stays unchanged (14 expansions, 14 config ids).
P07 asks T02 to cover gazebo and real at mast_1300 too, so those two expansions
run through check_urdf as labelled extras next to the planar ones (19 in all).

Assisted-by: Claude Code
Signed-off-by: Tushar Goel <Slash8860300674@gmail.com>

* docs(description): the config id's pin fallback, T02's extras, and the gripper interface limitation

The README documents where the upstream commit comes from and the two T02 extra
groups. The evidence report's limitations now say that the gripper controllers
are the deprecated position_controllers type on purpose: its replacement serves
ParallelGripperCommand, which would decide manipulation#11 / ADR-009 point 4.

Assisted-by: Claude Code
Signed-off-by: Tushar Goel <Slash8860300674@gmail.com>

* docs: CHANGELOG entries for the pin fallback, the T02 extras, .gitattributes and the gripper type

Assisted-by: Claude Code
Signed-off-by: Tushar Goel <Slash8860300674@gmail.com>

* feat(description): T10 prints the limit, the F2S vehicle estimate and a computed placeholder caveat

After the modelled total, T10 now reports the gross_mass_limit it compared against and
the F2S vehicle estimate (93 kg), each with its source and status from datums.yaml, and
the words "per-link masses still placeholders" if and only if a reported group draws a
mass from a datum whose status is placeholder. The clause is computed on every run
(MASS_DATUMS names the datums, and a test checks the xacro still reads them), so it
disappears when real masses land. Tests cover it appearing on the current tree and not
appearing on a synthetic set in which every mass datum is verified.

The F2S estimate is a new report_only datum, f2s_vehicle_mass_estimate (source f2s,
status provisional), so 93 is not written into the reporter or a test. datums revision
2026-10-08.e.

Assisted-by: Claude Code
Signed-off-by: Tushar Goel <Slash8860300674@gmail.com>

* feat(description): C02 checks upstream_pins.yaml against the upstream checkout

config/upstream_pins.yaml is the config id's fallback when src/upstream is absent, so it
is only useful while it equals the commit a real checkout is at. Nothing compared the two
when the checkout was there: C01's comparison passed vacuously without one, and with one
it was a test assertion, not a result in the evidence report.

C02 compares the pin with the HEAD of a clean checkout: equal is PASS, different is FAIL
naming both hashes, a dirty checkout or a missing pin is FAIL, and no checkout is SKIP
with the reason, which says it is the only legitimate SKIP in this tree. It compares with
the checkout, never with upstream's tip, so a pin held behind upstream is not drift. An
all-digit hash that YAML would read as a number is a FAIL, not a silent mismatch.

The comparison moves out of C01 into C02 (C01 keeps the format and the baseline pin).
The three outcomes are tested on synthetic checkouts; C02's own result is recorded in the
evidence report through a sidecar.

Assisted-by: Claude Code
Signed-off-by: Tushar Goel <Slash8860300674@gmail.com>

* docs(control): the gripper deprecation note states the five things in order

The README note now says, in this order: which controller and action type are in use;
that t

File: ros2/src/openamrobot_upperbody_description/urdf/openamrobot_upperbody.xacro (robot description, xacro)
@@ -34,8 +34,13 @@
                      horizontal plane (the column top at lift 0) and centred laterally;
                      center_x is from the column axis (datum adapter_plate_section).
+    datums           '' (none): no equipment. The parsed datums.yaml: the P-03 item 24 equipment
+                     of upper_body_equipment.xacro (placeholder geometry, fixed joints only) on
+                     arm_profile_link, adapter_plate_link and lift_column_base_link. Needs
+                     adapter_plate (the flag rod hangs from it); the combined robot passes both.
 -->
 <robot xmlns:xacro="http://www.ros.org/wiki/xacro">
+  <xacro:include filename="$(find openamrobot_upperbody_description)/urdf/upper_body_equipment.xacro"/>
   <xacro:macro name="openamrobot_upperbody"
-      params="parent column base_plate head_pitch base_tilt column_axis_x_bp000 emit_arm_mounts:=true column_inertial:='' column_geometry:='' adapter_plate:=''">
+      params="parent column base_plate head_pitch base_tilt column_axis_x_bp000 emit_arm_mounts:=true column_inertial:='' column_geometry:='' adapter_plate:='' datums:=''">
     <xacro:property name="cfg" lazy_eval="false"
         value="${xacro.load_yaml('$(find openamrobot_upperbody_description)/config/upperbody_configuration.yaml')}"/>
@@ -206,5 +211,14 @@
       <origin xyz="${mount['x_from_column_axis'] + lens['x_ahead_of_arm_mount']} ${lens['y']} ${mount['z_above_column_top'] + lens['z_above_arm_mount']}" rpy="0 0 0"/>
     </joint>
-    <link name="head_camera_link"/>
+    <!-- With the datums (combined robot): the ZED Mini body (upper_body_equipment.xacro); without: a frame, as before. -->
+    <xacro:if value="${datums == ''}">
+      <link name="head_camera_link"/>
+    </xacro:if>
+    <xacro:unless value="${datums == ''}">
+      <link name="head_camera_link">
+        <xacro:openamrobot_head_camera_body datums="${datums}"/>
+      </link>
+      <xacro:openamrobot_placeholder_gazebo_material link="head_camera_link"/>
+    </xacro:unless>
     <joint name="head_camera_pitch_joint" type="fixed">
       <parent link="head_camera_mount_link"/>
@@ -218,4 +232,11 @@
       <origin xyz="0 0 0" rpy="${-pi / 2} 0 ${-pi / 2}"/>
     </joint>
+    <!-- P-03 item 24 equipment (placeholder geometry, P-03 rev20.1 item 25 D8): upper_body_equipment.xacro. -->
+    <xacro:unless value="${datums == ''}">
+      <xacro:if value="${adapter_plate == ''}">
+        ${xacro.fatal("the item 24 equipment needs adapter_plate: the flag rod hangs from adapter_plate_link")}
+      </xacro:if>
+      <xacro:openamrobot_upper_body_equipment datums="${datums}" col="${col}" geo="${geo}"/>
+    </xacro:unless>
   </xacro:macro>
 </robot>
