Commit message: description, control: lift_joint position interface and lift_controller in mock and Gazebo (#17)
The simulated profiles (mock, gazebo) give lift_joint its own ros2_control system with a position
command interface and the DOLD V4 limits from two new datums (lift_max_effort_dold_v4_350 800 N,
lift_max_velocity_dold_v4_350 0.018 m/s; register LIFT, DOLD datasheet). lift_controller
(JointTrajectoryController) is spawned after joint_state_broadcaster with the arm controllers in
mock.launch.py and sim.launch.py. The real profile is unchanged: effort 0 velocity 0 and no
interface for the lift. T04, T14, T15, T16 and the spawner test follow the new hardware contract;
their real-profile assertions are kept.

Assisted-by: Claude Code
Signed-off-by: Alex Reznichenko <info@botshare.ai>

File: ros2/src/openamrobot_upperbody_description/urdf/combined_robot.xacro (robot description, xacro)
@@ -7,5 +7,5 @@
       -> lift_column_base_link                                  (option B, openamrobot_upperbody.xacro; datum column_axis_x_bp000)
            -> second_estop_link, lift_stop_sensor_{l1000,l1175,l1350}_link   (item 24 equipment, static: geometry only)
-           -> lift_joint (prismatic, 0..0.350 m, effort 0 velocity 0: no authority to command it) -> lift_carriage_link
+           -> lift_joint (prismatic, 0..0.350 m; mock/gazebo: 800 N, 0.018 m/s, planned; real: effort 0 velocity 0) -> lift_carriage_link
                 -> arm_profile_link -> getac_tablet_link, head_light_link          (P-03 item 24 equipment, upper_body_equipment.xacro)
                 -> adapter_plate_link -> lift_flag_rod_link -> lift_flag_link       (item 24)
@@ -19,6 +19,10 @@
   composition: the arms, the lift column's inertial (datums), the sensors on the wrists, ros2_control. No mast: the shoulder
   height is the joint position of lift_joint (calibration IDs L1000 / L1175 / L1350 are joint positions, not arguments).
-  ros2_control (ros2_control.xacro): arms only, none for the base and none for the lift. hardware_profile picks the arm plugin:
-  mock = mock_components/GenericSystem, gazebo = gz_ros2_control/GazeboSimSystem, real = openarm_hardware/OpenArmHW (ADR-003).
+  ros2_control (ros2_control.xacro): the arms, and the lift in the simulated profiles only; none for the base. hardware_profile picks the
+  arm plugin: mock = mock_components/GenericSystem, gazebo = gz_ros2_control/GazeboSimSystem, real = openarm_hardware/OpenArmHW (ADR-003).
+  The lift (issue #17): with mock and gazebo, lift_joint has its own <ros2_control> system (a position command interface, on the same
+  plugin as the arms) and carries the DOLD V4 limits (datums lift_max_effort_*, lift_max_velocity_*, register LIFT), so MoveIt plans it
+  and lift_controller follows it. With real it has neither: effort 0 velocity 0 and no command interface (the lift node firmware owns the
+  lift, CTL-017).
   Args: an unknown value for any arg fails expansion with the list of accepted values. column, base_plate, head_pitch and
   base_tilt are option B's configuration IDs; their accepted values and baseline are read from upperbody_configuration.yaml.
@@ -104,4 +108,17 @@
     ${xacro.fatal("column '" + column + "': retracted length is pending supplier data; this configuration cannot be built yet")}
   </xacro:if>
+  <!-- The lift's simulated limits (issue #17): the DOLD figures of the selected column, only where the lift has a controller (arm_package
+       openarm, hardware_profile mock or gazebo). Anywhere else lift_joint keeps effort 0 velocity 0. -->
+  <xacro:property name="lift_commanded" lazy_eval="false" value="${arm_package == 'openarm' and hardware_profile in ['mock', 'gazebo']}"/>
+  <xacro:property name="lift_motion_by_column" lazy_eval="false"
+                  value="${dict(dold_v4_350=dict(effort=dt['lift_max_effort_dold_v4_350']['value'], velocity=dt['lift_max_velocity_dold_v4_350']['value']))}"/>
+  <xacro:if value="${lift_commanded}">
+    <xacro:if value="${column not in lift_motion_by_column}">
+      ${xacro.fatal("column '" + column + "': no lift effort and velocity datums; the simulated lift cannot be built for it")}
+    </xacro:if>
+    <xacro:openamr_require_datum name="lift_max_effort_${column}" value="${lift_motion_by_column[column]['effort']}" owner="Alex (F2S)"/>
+    <xacro:openamr_require_datum name="lift_max_velocity_${column}" value="${lift_motion_by_column[column]['velocity']}" owner="Alex (F2S)"/>
+  </xacro:if>
+  <xacro:property name="lift_limits" lazy_eval="false" value="${lift_motion_by_column[column] if lift_commanded else ''}"/>
   <xacro:property name="lift_section" lazy_eval="false" value="${dt['lift_column_section']['value']}"/>
   <xacro:property name="lift_inner" lazy_eval="false" value="${dt['lift_inner_section']['value']}"/>
@@ -122,5 +139,5 @@
                                column_geometry="${dict(section_x=lift_section[0], section_y=lift_section[1], inner_x=lift_inner[0], inner_y=lift_inner[1])}"
                                adapter_plate="${dict(size_x=plate_section[0], size_y=plate_section[1], center_x=-lift_section[0] / 2 + plate_section[0] / 2)}"
-                               datums="${datums}"/>
+                               datums="${datums}" lift_limits="${lift_limits}"/>
   <!-- so101: stub only. A9 (Jonathan) owns everything below so101_mount_link; nothing else is emitted for it here.
        none: the upper body only. -->
@@ -165,7 +182,9 @@
     <xacro:include filename="$(find openamrobot_upperbody_description)/urdf/upper_sensors.xacro"/>
     <xacro:openamr_upper_sensors datums="${datums}"/>
-    <!-- Arms only, and only here: so101 and none get no ros2_control. Needs the arm joints emitted above. -->
+    <!-- Only here: so101 and none get no ros2_control. Needs the arm joints emitted above. -->
     <xacro:include filename="$(find openamrobot_upperbody_description)/urdf/ros2_control.xacro"/>
     <xacro:openamr_arm_ros2_control hardware_profile="${hardware_profile}" controllers_file="${controllers_file}"/>
+    <!-- The lift: mock and gazebo only (issue #17); real gets none. -->
+    <xacro:openamr_lift_ros2_control hardware_profile="${hardware_profile}"/>
   </xacro:if>
 </robot>

File: ros2/src/openamrobot_upperbody_description/urdf/openamrobot_upperbody.xacro (robot description, xacro)
@@ -34,4 +34,8 @@
                      horizontal plane (the column top at lift 0) and centred laterally;
                      center_x is from the column axis (datum adapter_plate_section).
+    lift_limits      '' (none): lift_joint carries effort 0 velocity 0, so the model cannot be used to command the
+                     lift (the default, and what the real profile keeps). A dict {effort, velocity}: those limits on
+                     lift_joint; the combined robot passes the DOLD figures (datums lift_max_effort_*, lift_max_velocity_*)
+                     for the simulated profiles (mock, gazebo) only, where the lift is a planned joint with a controller.
     datums           '' (none): no equipment. The parsed datums.yaml: the P-03 item 24 equipment
                      of upper_body_equipment.xacro (placeholder geometry, fixed joints only) on
@@ -42,5 +46,5 @@
   <xacro:include filename="$(find openamrobot_upperbody_description)/urdf/upper_body_equipment.xacro"/>
   <xacro:macro name="openamrobot_upperbody"
-      params="parent column base_plate head_pitch base_tilt column_axis_x_bp000 emit_arm_mounts:=true column_inertial:='' column_geometry:='' adapter_plate:='' datums:=''">
+      params="parent column base_plate head_pitch base_tilt column_axis_x_bp000 emit_arm_mounts:=true column_inertial:='' column_geometry:='' adapter_plate:='' datums:='' lift_limits:=''">
     <xacro:property name="cfg" lazy_eval="false"
         value="${xacro.load_yaml('$(find openamrobot_upperbody_description)/config/upperbody_configuration.yaml')}"/>
@@ -116,6 +120,7 @@
     </joint>
     <!-- Lift carriage: origin on the column axis at the column top. The lift
-         height is joint state. Effort and velocity limits are pending: they are
-         set to 0 so the model cannot be used to command the lift. -->
+         height is joint state. Effort and velocity are 0 unless lift_limits is
+         given (the combined robot's simulated profiles): with 0 the model cannot
+         be used to command the lift. -->
     <xacro:if value="${column_geometry == ''}">
       <link name="lift_carriage_link"/>
@@ -140,5 +145,10 @@
       <origin xyz="0 0 ${col['retracted_length']}" rpy="0 0 0"/>
       <axis xyz="0 0 1"/>
-      <limit lower="0.0" upper="${col['stroke']}" effort="0.0" velocity="0.0"/>
+      <xacro:if value="${lift_limits == ''}">
+        <limit lower="0.0" upper="${col['stroke']}" effort="0.0" velocity="0.0"/>
+      </xacro:if>
+      <xacro:unless value="${lift_limits == ''}">
+        <limit lower="0.0" upper="${col['stroke']}" effort="${lift_limits['effort']}" velocity="${lift_limits['velocity']}"/>
+      </xacro:unless>
     </joint>
     <!-- Adapter plate (P-03 rev19.6 item 18): its own link, carried by the carriage, under the arm profile. Its joint is at the box centre and

File: ros2/src/openamrobot_upperbody_description/urdf/ros2_control.xacro (robot description, xacro)
@@ -11,4 +11,9 @@
   finger-mimic multiplier file, same arm_type / ee_type / prefixes. The CAN interfaces and can_fd are not passed, so
   they take upstream's defaults, as they do in that file. Only use_fake_hardware differs: it follows the profile.
+  openamr_lift_ros2_control(hardware_profile) (issue #17): lift_joint in its own system, simulated profiles only.
+      mock    openamr_lift_mock    -> mock_components/GenericSystem
+      gazebo  openamr_lift_gazebo  -> gz_ros2_control/GazeboSimSystem (the same model plugin as the arms loads every system)
+      real    nothing: no command interface, no state interface. The lift node firmware owns the lift (CTL-017); the register LIFT
+              rule (lift motion only in the stowed or carry pose with the base stopped) is enforced there, not by this repository.
   The arm joints are openarm_{left,right}_joint1..7 and openarm_{left,right}_finger_joint1. Upstream leaves
   openarm_*_finger_joint2 out of <ros2_control> (its declaration is commented out in the macro); the URDF <mimic> on
@@ -113,3 +118,28 @@
     </xacro:if>
   </xacro:macro>
+  <!-- The lift (issue #17): a position command interface (lift_controller, a JointTrajectoryController, commands position) and position
+       and velocity state, starting at 0 (calibration stop L1000). Simulated profiles only; `real` declares nothing. -->
+  <xacro:macro name="openamr_lift_ros2_control" params="hardware_profile">
+    <xacro:if value="${hardware_profile in ['mock', 'gazebo']}">
+      <ros2_control name="openamr_lift_${hardware_profile}" type="system">
+        <hardware>
+          <xacro:if value="${hardware_profile == 'mock'}">
+            <plugin>mock_components/GenericSystem</plugin>
+          </xacro:if>
+          <xacro:if value="${hardware_profile == 'gazebo'}">
+            <plugin>gz_ros2_control/GazeboSimSystem</plugin>
+          </xacro:if>
+        </hardware>
+        <joint name="lift_joint">
+          <command_interface name="position"/>
+          <state_interface name="position">
+            <param name="initial_value">0.0</param>
+          </state_interface>
+          <state_interface name="velocity">
+            <param name="initial_value">0.0</param>
+          </state_interface>
+        </joint>
+      </ros2_control>
+    </xacro:if>
+  </xacro:macro>
 </robot>
